Commit message: Create fixed joint with colors

File: urdf/rover.urdf (robot description, URDF)
Before this commit: robot myfirst, 1 links, 0 joints
Links:
- added link pi_link; visual box size=0.12 0.15 0.05
- link base_link: geometry visual box size=0.14 0.2 0.01
Joints:
- added joint base_to_pi: type fixed, parent base_link, child pi_link, origin xyz=0 0 0

Commit message: Created motor link

File: urdf/rover.urdf (robot description, URDF)
Before this commit: robot rover, 2 links, 1 joints
Links:
- added link left_motor; visual box size=0.02 0.065 0.02
Joints:
- added joint base_to_left_motor: type fixed, parent base_link, child left_motor, origin xyz=-0.06 0 -0.015
- joint base_to_pi: origin xyz=0 0 0 -> xyz=0 0 0.03

File: urdf/rover.urdf.xacro (robot description, xacro)
@@ -4,6 +4,6 @@
     <color rgba="${245/255} ${222/255} ${179/255} 1"/>
   </material>
-  <material name="green">
-    <color rgba="0 0.8 0 1"/>
+  <material name="yellow">
+    <color rgba="0.8 0.8 0 1"/>
   </material>
   <link name="base_link">
@@ -20,6 +20,6 @@
         <box size="0.12 0.15 0.05"/>
       </geometry>
-      <origin rpy="0 0 0" xyz="0 0 0.03"/>
-      <material name="green"/>
+      <origin rpy="0 0 0" xyz="0 0 0"/>
+      <material name="tan"/>
     </visual>
   </link>
@@ -27,5 +27,22 @@
     <parent link="base_link"/>
     <child link="pi_link"/>
-    <origin xyz="0 0 0"/>
+    <origin xyz="0 0 0.03"/>
   </joint>
+  <xacro:macro name="wheel" params="prefix reflect">
+    <link name="${prefix}_motor">
+      <visual>
+        <geometry>
+          <box size="0.02 0.065 0.02"/>
+        </geometry>
+        <origin rpy="0 0 0" xyz="0 0 0"/>
+      	<material name="yellow"/>
+      </visual>
+    </link>
+    <joint name="base_to_${prefix}_motor" type="fixed">
+      <parent link="base_link"/>
+      <child link="${prefix}_motor"/>
+      <origin xyz="${reflect*0.06} 0 ${reflect*0.015}"/>
+    </joint>
+  </xacro:macro>
+  <xacro:wheel prefix="left" reflect="-1"/>
 </robot>
