Commit message: Created right motor and adjusted y position of motors

File: urdf/rover.urdf.xacro (robot description, xacro)
@@ -42,7 +42,8 @@
       <parent link="base_link"/>
       <child link="${prefix}_motor"/>
-      <origin xyz="${reflect*0.06} 0 ${reflect*0.015}"/>
+      <origin xyz="${reflect*0.06} 0.02 -0.015"/>
     </joint>
   </xacro:macro>
   <xacro:wheel prefix="left" reflect="-1"/>
+  <xacro:wheel prefix="right" reflect="1"/>
 </robot>

Commit message: Added wheels as fixed joints

File: urdf/rover.urdf.xacro (robot description, xacro)
@@ -1,4 +1,5 @@
 <?xml version="1.0"?>
 <robot xmlns:xacro="http://www.ros.org/wiki/xacro" name="rover">
+  <xacro:property name="pi" value="3.1415"/>
   <material name="tan">
     <color rgba="${245/255} ${222/255} ${179/255} 1"/>
@@ -7,8 +8,11 @@
     <color rgba="0.8 0.8 0 1"/>
   </material>
+  <material name="black">
+    <color rgba="0 0 0 1"/>
+  </material>
   <link name="base_link">
     <visual>
       <geometry>
-        <box size="0.14 0.2 0.01"/>
+        <box size="0.14 0.20 0.01"/>
       </geometry>
       <material name="tan"/>
@@ -42,5 +46,19 @@
       <parent link="base_link"/>
       <child link="${prefix}_motor"/>
-      <origin xyz="${reflect*0.06} 0.02 -0.015"/>
+      <origin xyz="${reflect*0.06} 0.01 -0.015"/>
+    </joint>
+    <link name="${prefix}_wheel">
+      <visual>
+        <geometry>
+          <cylinder length="0.027" radius="0.0325"/>
+        </geometry>
+        <origin xyz="0 0 0" rpy="0 ${pi/2} 0"/>
+        <material name="black"/>
+      </visual>
+    </link>
+    <joint name="${prefix}_motor_to_wheel" type="fixed">
+      <parent link="${prefix}_motor"/>
+      <child link="${prefix}_wheel"/>
+      <origin xyz="${reflect*0.025} 0.02 0"/>
     </joint>
   </xacro:macro>

Commit message: Added laser_frame link

File: urdf/rover.urdf.xacro (robot description, xacro)
@@ -33,4 +33,18 @@
     <origin xyz="0 0 0.03"/>
   </joint>
+  <link name="laser_frame">
+    <visual>
+      <geometry>
+        <cylinder length="0.03" radius="0.035"/>
+      </geometry>
+      <origin rpy="0 0 0" xyz="0 0 0"/>
+      <material name="tan"/>
+    </visual>
+  </link>
+  <joint name="pi_to_lidar" type="fixed">
+    <parent link="pi_link"/>
+    <child link="laser_frame"/>
+    <origin xyz="0 0.02 0.035"/>
+  </joint>
   <xacro:macro name="wheel" params="prefix reflect">
     <link name="${prefix}_motor">

Commit message: Make wheels continuous joint

File: urdf/rover.urdf.xacro (robot description, xacro)
@@ -71,7 +71,8 @@
       </visual>
     </link>
-    <joint name="${prefix}_motor_to_wheel" type="fixed">
+    <joint name="${prefix}_motor_to_wheel" type="continuous">
       <parent link="${prefix}_motor"/>
       <child link="${prefix}_wheel"/>
+      <axis xyz="1 0 0"/>
       <origin xyz="${reflect*0.025} 0.02 0"/>
     </joint>

Commit message: Moved wheel to separate xacro file

File: urdf/rover.urdf.xacro (robot description, xacro)
@@ -1,13 +1,8 @@
 <?xml version="1.0"?>
 <robot xmlns:xacro="http://www.ros.org/wiki/xacro" name="rover">
+  <xacro:include filename="$(find rover)/urdf/wheel.urdf.xacro"/>
   <xacro:property name="pi" value="3.1415"/>
   <material name="tan">
     <color rgba="${245/255} ${222/255} ${179/255} 1"/>
-  </material>
-  <material name="yellow">
-    <color rgba="0.8 0.8 0 1"/>
-  </material>
-  <material name="black">
-    <color rgba="0 0 0 1"/>
   </material>
   <link name="base_link">
@@ -47,35 +42,4 @@
     <origin xyz="0 0.02 0.035"/>
   </joint>
-  <xacro:macro name="wheel" params="prefix reflect">
-    <link name="${prefix}_motor">
-      <visual>
-        <geometry>
-          <box size="0.02 0.065 0.02"/>
-        </geometry>
-        <origin rpy="0 0 0" xyz="0 0 0"/>
-      	<material name="yellow"/>
-      </visual>
-    </link>
-    <joint name="base_to_${prefix}_motor" type="fixed">
-      <parent link="base_link"/>
-      <child link="${prefix}_motor"/>
-      <origin xyz="${reflect*0.06} 0.01 -0.015"/>
-    </joint>
-    <link name="${prefix}_wheel">
-      <visual>
-        <geometry>
-          <cylinder length="0.027" radius="0.0325"/>
-        </geometry>
-        <origin xyz="0 0 0" rpy="0 ${pi/2} 0"/>
-        <material name="black"/>
-      </visual>
-    </link>
-    <joint name="${prefix}_motor_to_wheel" type="continuous">
-      <parent link="${prefix}_motor"/>
-      <child link="${prefix}_wheel"/>
-      <axis xyz="1 0 0"/>
-      <origin xyz="${reflect*0.025} 0.02 0"/>
-    </joint>
-  </xacro:macro>
   <xacro:wheel prefix="left" reflect="-1"/>
   <xacro:wheel prefix="right" reflect="1"/>

Commit message: Added caster support link

File: urdf/rover.urdf.xacro (robot description, xacro)
@@ -2,5 +2,4 @@
 <robot xmlns:xacro="http://www.ros.org/wiki/xacro" name="rover">
   <xacro:include filename="$(find rover)/urdf/wheel.urdf.xacro"/>
-  <xacro:property name="pi" value="3.1415"/>
   <material name="tan">
     <color rgba="${245/255} ${222/255} ${179/255} 1"/>
@@ -42,4 +41,18 @@
     <origin xyz="0 0.02 0.035"/>
   </joint>
+  <link name="caster_support">
+    <visual>
+      <geometry>
+        <box size="0.02 0.02 0.03"/>
+      </geometry>
+      <origin rpy="0 0 0" xyz="0 0 0"/>
+      <material name="tan"/>
+    </visual>
+  </link>
+  <joint name="base_to_caster_support" type="fixed">
+    <parent link="base_link"/>
+    <child link="caster_support"/>
+    <origin xyz="0 -0.07 -0.02"/>
+  </joint>
   <xacro:wheel prefix="left" reflect="-1"/>
   <xacro:wheel prefix="right" reflect="1"/>

Commit message: Created caster wheel as fixed joint

File: urdf/rover.urdf.xacro (robot description, xacro)
@@ -55,4 +55,18 @@
     <origin xyz="0 -0.07 -0.02"/>
   </joint>
+  <link name="caster_wheel">
+    <visual>
+      <geometry>
+        <sphere radius="0.01"/>
+      </geometry>
+      <origin rpy="0 0 0" xyz="0 0 0"/>
+      <material name="black"/>
+    </visual>
+  </link>
+  <joint name="caster_support_to_wheel" type="fixed">
+    <parent link="caster_support"/>
+    <child link="caster_wheel"/>
+    <origin xyz="0 0 -0.02"/>
+  </joint>
   <xacro:wheel prefix="left" reflect="-1"/>
   <xacro:wheel prefix="right" reflect="1"/>

Commit message: Leveled wheels

File: urdf/rover.urdf.xacro (robot description, xacro)
@@ -2,4 +2,7 @@
 <robot xmlns:xacro="http://www.ros.org/wiki/xacro" name="rover">
   <xacro:include filename="$(find rover)/urdf/wheel.urdf.xacro"/>
+  <xacro:property name="base_d" value="0.01"/>
+  <xacro:property name="caster_r" value="0.01"/>
+  <xacro:property name="csupp_d" value="${wheel_r + 0.5*motor_d - 1.5*caster_r}"/>
   <material name="tan">
     <color rgba="${245/255} ${222/255} ${179/255} 1"/>
@@ -13,4 +16,18 @@
     </visual>
   </link>
+  <link name="base_footprint">
+    <visual>
+      <geometry>
+        <box size="0.001 0.001 0.001"/>
+      </geometry>
+      <origin xyz="0 0 0" rpy="0 0 0"/>
+      <material name="tan"/>
+    </visual>
+  </link>
+  <joint name="base_to_footprint" type="fixed">
+    <parent link="base_link"/>
+    <child link="base_footprint"/>
+    <origin xyz="0 0 ${-(0.5*base_d + 0.5*motor_d + wheel_r)}"/>
+  </joint>
   <link name="pi_link">
     <visual>
@@ -44,5 +61,5 @@
     <visual>
       <geometry>
-        <box size="0.02 0.02 0.03"/>
+        <box size="0.02 0.02 ${csupp_d}"/>
       </geometry>
       <origin rpy="0 0 0" xyz="0 0 0"/>
@@ -53,10 +70,10 @@
     <parent link="base_link"/>
     <child link="caster_support"/>
-    <origin xyz="0 -0.07 -0.02"/>
+    <origin xyz="0 -0.07 ${-(0.5*csupp_d + 0.5*base_d)}"/>
   </joint>
   <link name="caster_wheel">
     <visual>
       <geometry>
-        <sphere radius="0.01"/>
+        <sphere radius="${caster_r}"/>
       </geometry>
       <origin rpy="0 0 0" xyz="0 0 0"/>
@@ -67,5 +84,5 @@
     <parent link="caster_support"/>
     <child link="caster_wheel"/>
-    <origin xyz="0 0 -0.02"/>
+    <origin xyz="0 0 ${-(0.5*csupp_d + 0.5*caster_r)}"/>
   </joint>
   <xacro:wheel prefix="left" reflect="-1"/>

File: urdf/wheel.urdf.xacro (robot description, xacro)
@@ -2,4 +2,6 @@
 <robot xmlns:xacro="http://www.ros.org/wiki/xacro" name="wheel">
   <xacro:property name="pi" value="3.1415"/>
+  <xacro:property name="motor_d" value="0.02"/>
+  <xacro:property name="wheel_r" value="0.0325"/>
   <material name="yellow">
     <color rgba="0.8 0.8 0 1"/>
@@ -12,5 +14,5 @@
       <visual>
         <geometry>
-          <box size="0.02 0.065 0.02"/>
+          <box size="0.02 0.065 ${motor_d}"/>
         </geometry>
         <origin rpy="0 0 0" xyz="0 0 0"/>
@@ -26,5 +28,5 @@
       <visual>
         <geometry>
-          <cylinder length="0.027" radius="0.0325"/>
+          <cylinder length="0.027" radius="${wheel_r}"/>
         </geometry>
         <origin xyz="0 0 0" rpy="0 ${pi/2} 0"/>

Commit message: Adding collision and inertia to base components

File: urdf/rover.urdf.xacro (robot description, xacro)
@@ -2,14 +2,28 @@
 <robot xmlns:xacro="http://www.ros.org/wiki/xacro" name="rover">
   <xacro:include filename="$(find rover)/urdf/colors.xacro"/>
+  <xacro:include filename="$(find rover)/urdf/inertia.xacro"/>
   <xacro:include filename="$(find rover)/urdf/motor_wheel.xacro"/>
   <xacro:include filename="$(find rover)/urdf/caster_wheel.xacro"/>
   <xacro:property name="base_d" value="0.01"/>
+  <xacro:property name="bl_m" value="0.1"/>
+  <xacro:property name="bl_w" value="0.14"/>
+  <xacro:property name="bl_h" value="0.20"/>
+  <xacro:property name="bl_d" value="0.01"/>
   <link name="base_link">
     <visual>
       <geometry>
-        <box size="0.14 0.20 0.01"/>
+        <box size="${bl_w} ${bl_h} ${bl_d}"/>
       </geometry>
       <material name="tan"/>
     </visual>
+    <collision>
+      <geometry>
+        <box size="${bl_w} ${bl_h} ${bl_d}"/>
+      </geometry>
+    </collision>
+    <inertial>
+      <mass value="${bl_m}"/>
+      <xacro:cuboid_i m="${bl_m}" w="${bl_w}" h="${bl_h}" d="${bl_d}"/>
+    </inertial>
   </link>
   <link name="base_footprint">
@@ -27,12 +41,25 @@
     <origin xyz="0 0 ${-(0.5*base_d + 0.5*motor_d + wheel_r)}"/>
   </joint>
+  <xacro:property name="p_m" value="0.4"/>
+  <xacro:property name="p_w" value="0.12"/>
+  <xacro:property name="p_h" value="0.15"/>
+  <xacro:property name="p_d" value="0.05"/>
   <link name="pi_link">
     <visual>
       <geometry>
-        <box size="0.12 0.15 0.05"/>
+        <box size="${p_w} ${p_h} ${p_d}"/>
       </geometry>
       <origin rpy="0 0 0" xyz="0 0 0"/>
       <material name="tan"/>
     </visual>
+    <collision>
+      <geometry>
+        <box size="${p_w} ${p_h} ${p_d}"/>
+      </geometry>
+    </collision>
+    <inertial>
+      <mass value="${p_m}"/>
+      <xacro:cuboid_i m="${p_m}" w="${p_w}" h="${p_h}" d="${p_d}"/>
+    </inertial>
   </link>
   <joint name="base_to_pi" type="fixed">
@@ -41,12 +68,24 @@
     <origin xyz="0 0 0.03"/>
   </joint>
+  <xacro:property name="l_m" value="0.2"/>
+  <xacro:property name="l_l" value="0.03"/>
+  <xacro:property name="l_r" value="0.035"/>
   <link name="laser_frame">
     <visual>
       <geometry>
-        <cylinder length="0.03" radius="0.035"/>
+        <cylinder length="${l_l}" radius="${l_r}"/>
       </geometry>
       <origin rpy="0 0 0" xyz="0 0 0"/>
       <material name="tan"/>
     </visual>
+    <collision>
+      <geometry>
+        <cylinder length="${l_l}" radius="${l_r}"/>
+      </geometry>
+    </collision>
+    <inertial>
+      <mass value="${l_m}"/>
+      <xacro:cylinder_i m="${l_m}" l="${l_l}" r="${l_r}"/>
+    </inertial>
   </link>
   <joint name="pi_to_lidar" type="fixed">
