Commit message: Moved colors to separate xacro

File: urdf/caster_wheel.xacro (robot description, xacro)
@@ -3,7 +3,4 @@
   <xacro:property name="caster_r" value="0.01"/>
   <xacro:property name="csupp_d" value="${wheel_r + 0.5*motor_d - 1.5*caster_r}"/>
-  <material name="tan">
-    <color rgba="${245/255} ${222/255} ${179/255} 1"/>
-  </material>
   <link name="caster_support">
     <visual>

File: urdf/motor_wheel.xacro (robot description, xacro)
@@ -4,10 +4,4 @@
   <xacro:property name="motor_d" value="0.02"/>
   <xacro:property name="wheel_r" value="0.0325"/>
-  <material name="yellow">
-    <color rgba="0.8 0.8 0 1"/>
-  </material>
-  <material name="black">
-    <color rgba="0 0 0 1"/>
-  </material>
   <xacro:macro name="motorwheel" params="prefix reflect">
     <link name="${prefix}_motor">

File: urdf/rover.urdf.xacro (robot description, xacro)
@@ -1,4 +1,5 @@
 <?xml version="1.0"?>
 <robot xmlns:xacro="http://www.ros.org/wiki/xacro" name="rover">
+  <xacro:include filename="$(find rover)/urdf/colors.xacro"/>
   <xacro:include filename="$(find rover)/urdf/motor_wheel.xacro"/>
   <xacro:include filename="$(find rover)/urdf/caster_wheel.xacro"/>

Commit message: Added collision and inertials to caster links

File: urdf/caster_wheel.xacro (robot description, xacro)
@@ -1,33 +1,55 @@
 <?xml version="1.0"?>
 <robot xmlns:xacro="http://www.ros.org/wiki/xacro" name="casterwheel">
-  <xacro:property name="caster_r" value="0.01"/>
-  <xacro:property name="csupp_d" value="${wheel_r + 0.5*motor_d - 1.5*caster_r}"/>
+  <xacro:property name="cs_m" value="0.05"/>
+  <xacro:property name="cs_w" value="0.02"/>
+  <xacro:property name="cs_h" value="0.02"/>
+  <xacro:property name="cs_d" value="${wheel_r + 0.5*motor_d - 1.5*cw_r}"/>
   <link name="caster_support">
     <visual>
       <geometry>
-        <box size="0.02 0.02 ${csupp_d}"/>
+        <box size="${cs_w} ${cs_h} ${cs_d}"/>
       </geometry>
       <origin rpy="0 0 0" xyz="0 0 0"/>
       <material name="tan"/>
     </visual>
+    <collision>
+      <geometry>
+        <box size="${cs_w} ${cs_h} ${cs_d}"/>
+      </geometry>
+    </collision>
+    <inertial>
+      <mass value="${cs_m}"/>
+      <xacro:cuboid_i m="${cs_m}" w="${cs_w}" h="${cs_h}" d="${cs_d}"/>
+    </inertial>
   </link>
   <joint name="base_to_caster_support" type="fixed">
     <parent link="base_link"/>
     <child link="caster_support"/>
-    <origin xyz="0 -0.07 ${-(0.5*csupp_d + 0.5*base_d)}"/>
+    <origin xyz="0 -0.07 ${-(0.5*cs_d + 0.5*base_d)}"/>
   </joint>
+  <xacro:property name="cw_m" value="0.05"/>
+  <xacro:property name="cw_r" value="0.01"/>
   <link name="caster_wheel">
     <visual>
       <geometry>
-        <sphere radius="${caster_r}"/>
+        <sphere radius="${cw_r}"/>
       </geometry>
       <origin rpy="0 0 0" xyz="0 0 0"/>
       <material name="black"/>
     </visual>
+    <collision>
+      <geometry>
+        <sphere radius="${cw_r}"/>
+      </geometry>
+    </collision>
+    <inertial>
+      <mass value="${cw_m}"/>
+      <xacro:sphere_i m="${cw_m}" r="${cw_r}"/>
+    </inertial>
   </link>
   <joint name="caster_support_to_wheel" type="fixed">
     <parent link="caster_support"/>
     <child link="caster_wheel"/>
-    <origin xyz="0 0 ${-(0.5*csupp_d + 0.5*caster_r)}"/>
+    <origin xyz="0 0 ${-(0.5*cs_d + 0.5*cw_r)}"/>
   </joint>
 </robot>

File: urdf/inertia.xacro (robot description, xacro)
@@ -7,3 +7,6 @@
     <inertia ixx="${(1/12)*m*(3*r*r+l*l)}" ixy="0.0" ixz="0.0" iyy="${(1/12)*m*(3*r*r+l*l)}" iyz="0.0" izz="${(1/2)*m*r*r}"/>
   </xacro:macro>
+  <xacro:macro name="sphere_i" params="m r">
+    <inertia ixx="${(2/5)*m*r*r}" ixy="0.0" ixz="0.0" iyy="${(2/5)*m*r*r}" iyz="0.0" izz="${(2/5)*m*r*r}"/>
+  </xacro:macro>
 </robot>

Commit message: Added collision and inertials to motor wheels

File: urdf/caster_wheel.xacro (robot description, xacro)
@@ -4,5 +4,5 @@
   <xacro:property name="cs_w" value="0.02"/>
   <xacro:property name="cs_h" value="0.02"/>
-  <xacro:property name="cs_d" value="${wheel_r + 0.5*motor_d - 1.5*cw_r}"/>
+  <xacro:property name="cs_d" value="${w_r + 0.5*m_d - 1.5*cw_r}"/>
   <link name="caster_support">
     <visual>

File: urdf/motor_wheel.xacro (robot description, xacro)
@@ -2,15 +2,29 @@
 <robot xmlns:xacro="http://www.ros.org/wiki/xacro" name="motorwheel">
   <xacro:property name="pi" value="3.1415"/>
-  <xacro:property name="motor_d" value="0.02"/>
-  <xacro:property name="wheel_r" value="0.0325"/>
+  <xacro:property name="m_m" value="0.02"/>
+  <xacro:property name="m_w" value="0.02"/>
+  <xacro:property name="m_h" value="0.065"/>
+  <xacro:property name="m_d" value="0.02"/>
+  <xacro:property name="w_m" value="0.01"/>
+  <xacro:property name="w_r" value="0.0325"/>
+  <xacro:property name="w_l" value="0.027"/>
   <xacro:macro name="motorwheel" params="prefix reflect">
     <link name="${prefix}_motor">
       <visual>
         <geometry>
-          <box size="0.02 0.065 ${motor_d}"/>
+          <box size="${m_w} ${m_h} ${m_d}"/>
         </geometry>
         <origin rpy="0 0 0" xyz="0 0 0"/>
       	<material name="yellow"/>
       </visual>
+      <collision>
+        <geometry>
+          <box size="${m_w} ${m_h} ${m_d}"/>
+        </geometry>
+      </collision>
+      <inertial>
+        <mass value="${m_m}"/>
+        <xacro:cuboid_i m="${m_m}" w="${m_w}" h="${m_h}" d="${m_d}"/>
+      </inertial>
     </link>
     <joint name="base_to_${prefix}_motor" type="fixed">
@@ -22,9 +36,18 @@
       <visual>
         <geometry>
-          <cylinder length="0.027" radius="${wheel_r}"/>
+          <cylinder length="${w_l}" radius="${w_r}"/>
         </geometry>
         <origin xyz="0 0 0" rpy="0 ${pi/2} 0"/>
         <material name="black"/>
       </visual>
+      <collision>
+         <geometry>
+           <cylinder length="${w_l}" radius="${w_r}"/>
+         </geometry>
+      </collision>
+      <inertial>
+        <mass value="${w_m}"/>
+        <xacro:cylinder_i m="${w_m}" l="${w_l}" r="${w_r}"/>
+      </inertial>
     </link>
     <joint name="${prefix}_motor_to_wheel" type="continuous">

File: urdf/rover.urdf.xacro (robot description, xacro)
@@ -39,5 +39,5 @@
     <parent link="base_link"/>
     <child link="base_footprint"/>
-    <origin xyz="0 0 ${-(0.5*base_d + 0.5*motor_d + wheel_r)}"/>
+    <origin xyz="0 0 ${-(0.5*base_d + 0.5*m_d + w_r)}"/>
   </joint>
   <xacro:property name="p_m" value="0.4"/>

Commit message: Add macro to casterwheel.xacro

File: urdf/caster_wheel.xacro (robot description, xacro)
@@ -1,55 +1,57 @@
 <?xml version="1.0"?>
 <robot xmlns:xacro="http://www.ros.org/wiki/xacro" name="casterwheel">
-  <xacro:property name="cs_m" value="0.05"/>
-  <xacro:property name="cs_w" value="0.02"/>
-  <xacro:property name="cs_h" value="0.02"/>
-  <xacro:property name="cs_d" value="${w_r + 0.5*m_d - 1.5*cw_r}"/>
-  <link name="caster_support">
-    <visual>
-      <geometry>
-        <box size="${cs_w} ${cs_h} ${cs_d}"/>
-      </geometry>
-      <origin rpy="0 0 0" xyz="0 0 0"/>
-      <material name="tan"/>
-    </visual>
-    <collision>
-      <geometry>
-        <box size="${cs_w} ${cs_h} ${cs_d}"/>
-      </geometry>
-    </collision>
-    <inertial>
-      <mass value="${cs_m}"/>
-      <xacro:cuboid_i m="${cs_m}" w="${cs_w}" h="${cs_h}" d="${cs_d}"/>
-    </inertial>
-  </link>
-  <joint name="base_to_caster_support" type="fixed">
-    <parent link="base_link"/>
-    <child link="caster_support"/>
-    <origin xyz="0 -0.07 ${-(0.5*cs_d + 0.5*base_d)}"/>
-  </joint>
-  <xacro:property name="cw_m" value="0.05"/>
-  <xacro:property name="cw_r" value="0.01"/>
-  <link name="caster_wheel">
-    <visual>
-      <geometry>
-        <sphere radius="${cw_r}"/>
-      </geometry>
-      <origin rpy="0 0 0" xyz="0 0 0"/>
-      <material name="black"/>
-    </visual>
-    <collision>
-      <geometry>
-        <sphere radius="${cw_r}"/>
-      </geometry>
-    </collision>
-    <inertial>
-      <mass value="${cw_m}"/>
-      <xacro:sphere_i m="${cw_m}" r="${cw_r}"/>
-    </inertial>
-  </link>
-  <joint name="caster_support_to_wheel" type="fixed">
-    <parent link="caster_support"/>
-    <child link="caster_wheel"/>
-    <origin xyz="0 0 ${-(0.5*cs_d + 0.5*cw_r)}"/>
-  </joint>
+  <xacro:macro name="casterwheel" params="">
+		<xacro:property name="cs_m" value="0.05"/>
+		<xacro:property name="cs_w" value="0.02"/>
+		<xacro:property name="cs_h" value="0.02"/>
+		<xacro:property name="cs_d" value="${w_r + 0.5*m_d - 1.5*cw_r}"/>
+		<link name="caster_support">
+			<visual>
+				<geometry>
+					<box size="${cs_w} ${cs_h} ${cs_d}"/>
+				</geometry>
+				<origin rpy="0 0 0" xyz="0 0 0"/>
+				<material name="tan"/>
+			</visual>
+			<collision>
+				<geometry>
+					<box size="${cs_w} ${cs_h} ${cs_d}"/>
+				</geometry>
+			</collision>
+			<inertial>
+				<mass value="${cs_m}"/>
+				<xacro:cuboid_i m="${cs_m}" w="${cs_w}" h="${cs_h}" d="${cs_d}"/>
+			</inertial>
+		</link>
+		<joint name="base_to_caster_support" type="fixed">
+			<parent link="base_link"/>
+			<child link="caster_support"/>
+			<origin xyz="0 -0.07 ${-(0.5*cs_d + 0.5*base_d)}"/>
+		</joint>
+		<xacro:property name="cw_m" value="0.05"/>
+		<xacro:property name="cw_r" value="0.01"/>
+		<link name="caster_wheel">
+			<visual>
+				<geometry>
+					<sphere radius="${cw_r}"/>
+				</geometry>
+				<origin rpy="0 0 0" xyz="0 0 0"/>
+				<material name="black"/>
+			</visual>
+			<collision>
+				<geometry>
+					<sphere radius="${cw_r}"/>
+				</geometry>
+			</collision>
+			<inertial>
+				<mass value="${cw_m}"/>
+				<xacro:sphere_i m="${cw_m}" r="${cw_r}"/>
+			</inertial>
+		</link>
+		<joint name="caster_support_to_wheel" type="fixed">
+			<parent link="caster_support"/>
+			<child link="caster_wheel"/>
+			<origin xyz="0 0 ${-(0.5*cs_d + 0.5*cw_r)}"/>
+		</joint>
+	</xacro:macro>
 </robot>

Commit message: edit xacro files

File: urdf/caster_wheel.xacro (robot description, xacro)
@@ -1,9 +1,11 @@
 <?xml version="1.0"?>
 <robot xmlns:xacro="http://www.ros.org/wiki/xacro" name="casterwheel">
+  <xacro:property name="cs_m" value="0.05"/>
+  <xacro:property name="cs_w" value="0.02"/>
+  <xacro:property name="cs_h" value="0.02"/>
+  <xacro:property name="cs_d" value="${w_r + 0.5*m_d - 1.5*cw_r}"/>
+  <xacro:property name="cw_m" value="0.05"/>
+  <xacro:property name="cw_r" value="0.01"/>
   <xacro:macro name="casterwheel" params="">
-		<xacro:property name="cs_m" value="0.05"/>
-		<xacro:property name="cs_w" value="0.02"/>
-		<xacro:property name="cs_h" value="0.02"/>
-		<xacro:property name="cs_d" value="${w_r + 0.5*m_d - 1.5*cw_r}"/>
 		<link name="caster_support">
 			<visual>
@@ -29,6 +31,4 @@
 			<origin xyz="0 -0.07 ${-(0.5*cs_d + 0.5*base_d)}"/>
 		</joint>
-		<xacro:property name="cw_m" value="0.05"/>
-		<xacro:property name="cw_r" value="0.01"/>
 		<link name="caster_wheel">
 			<visual>

File: urdf/motor_wheel.xacro (robot description, xacro)
@@ -51,5 +51,5 @@
       </inertial>
     </link>
-    <joint name="${prefix}_motor_to_wheel" type="continuous">
+    <joint name="${prefix}_motor_to_wheel" type="fixed">
       <parent link="${prefix}_motor"/>
       <child link="${prefix}_wheel"/>

File: urdf/rover.urdf (robot description, URDF)
Before this commit: robot rover, 10 links, 9 joints
Links:
- removed link laser_frame
- added link laser_frame1, mass 0.2; collision cylinder length=0.03 radius=0.035; visual cylinder length=0.03 radius=0.035
Joints:
- joint left_motor_to_wheel: type continuous -> fixed
- joint pi_to_lidar: child laser_frame -> laser_frame1; origin xyz=0 0.02 0.035 -> xyz=0 0.02 0.035 rpy=0 0 1.57075
- joint right_motor_to_wheel: type continuous -> fixed

File: urdf/rover.urdf.xacro (robot description, xacro)
@@ -71,5 +71,5 @@
   <xacro:property name="l_l" value="0.03"/>
   <xacro:property name="l_r" value="0.035"/>
-  <link name="laser_frame">
+  <link name="laser_frame1">
     <visual>
       <geometry>
@@ -91,9 +91,9 @@
   <joint name="pi_to_lidar" type="fixed">
     <parent link="pi_link"/>
-    <child link="laser_frame"/>
-    <origin xyz="0 0.02 0.035"/>
+    <child link="laser_frame1"/>
+    <origin xyz="0 0.02 0.035" rpy="0 0 ${pi/2}"/>
   </joint>
-  <xacro:casterwheel />
   <xacro:motorwheel prefix="left" reflect="-1"/>
   <xacro:motorwheel prefix="right" reflect="1"/>
+  <xacro:casterwheel />
 </robot>
